File: smt_training pcb files/smt_training.kicad_sch (KiCad schematic)
At the start: 28 parts, among them J1 AU-Y1006-2, Q1 2N7002-7-F, SW1 PTS636SK25FSMTR LFS, SW2 PTS526SM15SMTR2 LFS, U1 SN74LVC1G08DBVR, U2 SN74LVC1G86DCKR, U3 LQFP64 IC, U4 NE555S-13

Commit message: Fixed Bypassed SW2; Added Soldermask to Back Icons; Updated Version Number
Connections:
- net +5V: now also SW2.2; no longer SW2.3
- net at R1.1, SW2.4, U1.2: now also SW2.3; no longer SW2.2
Changed lines of the file:
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@@
 	(title_block
 		(title "Soldering I + II Circuits")
-		(date "2025-10-17")
-		(rev "1")
+		(date "2025-11-26")
+		(rev "1.1")
 		(company "The Shop - Franklin W. Olin College of Engineering")
 		(comment 1 "Henry Tejada Deras + Emily Boyd")
@@
 	)
 	(junction
-		(at 142.24 69.85)
+		(at 78.74 72.39)
 		(diameter 0)
 		(color 0 0 0 0)
 	)
 	(junction
-		(at 82.55 142.24)
+		(at 142.24 69.85)
 		(diameter 0)
 		(color 0 0 0 0)
 	)
 	(junction
-		(at 138.43 69.85)
+		(at 82.55 142.24)
 		(diameter 0)
 		(color 0 0 0 0)
 	)
 	(junction
-		(at 82.55 133.35)
+		(at 138.43 69.85)
 		(diameter 0)
 		(color 0 0 0 0)
 	)
 	(junction
-		(at 78.74 72.39)
+		(at 82.55 133.35)
 		(diameter 0)
 		(color 0 0 0 0)
@@
 	(wire
 		(pts
-			(xy 78.74 71.12) (xy 78.74 72.39)
+			(xy 90.17 133.35) (xy 90.17 135.89)
 		)
 		(stroke
@@
 	(wire
 		(pts
-			(xy 90.17 133.35) (xy 90.17 135.89)
+			(xy 57.15 73.66) (xy 60.96 73.66)
 		)
 		(stroke
@@
 	(wire
 		(pts
-			(xy 59.69 73.66) (xy 60.96 73.66)
+			(xy 38.1 149.86) (xy 40.64 149.86)
 		)
 		(stroke
@@
 	(wire
 		(pts
-			(xy 38.1 149.86) (xy 40.64 149.86)
+			(xy 20.32 151.13) (xy 20.32 149.86)
 		)
 		(stroke
@@
 	(wire
 		(pts
-			(xy 20.32 151.13) (xy 20.32 149.86)
+			(xy 82.55 142.24) (xy 82.55 156.21)
 		)
 		(stroke
@@
 	(wire
 		(pts
-			(xy 82.55 142.24) (xy 82.55 156.21)
+			(xy 123.19 50.8) (xy 123.19 59.69)
 		)
 		(stroke
@@
 	(wire
 		(pts
-			(xy 123.19 50.8) (xy 123.19 59.69)
+			(xy 90.17 133.35) (xy 90.17 132.08)
 		)
 		(stroke
@@
 	(wire
 		(pts
-			(xy 90.17 133.35) (xy 90.17 132.08)
+			(xy 78.74 71.12) (xy 78.74 72.39)
 		)
 		(stroke
@@
 	(wire
 		(pts
-			(xy 135.89 96.52) (xy 138.43 96.52)
+			(xy 129.54 96.52) (xy 138.43 96.52)
 		)
 		(stroke
@@
 	(wire
 		(pts
-			(xy 73.66 134.62) (xy 73.66 133.35)
+			(xy 77.47 71.12) (xy 78.74 71.12)
 		)
 		(stroke
@@
 	(wire
 		(pts
-			(xy 15.24 142.24) (xy 43.18 142.24)
+			(xy 73.66 134.62) (xy 73.66 133.35)
 		)
 		(stroke
@@
 	(wire
 		(pts
-			(xy 73.66 133.35) (xy 74.93 133.35)
+			(xy 15.24 142.24) (xy 43.18 142.24)
 		)
 		(stroke
@@
 	(wire
 		(pts
-			(xy 82.55 142.24) (xy 73.66 142.24)
+			(xy 73.66 133.35) (xy 74.93 133.35)
 		)
 		(stroke
@@
 	(wire
 		(pts
-			(xy 43.18 149.86) (xy 43.18 156.21)
+			(xy 82.55 142.24) (xy 73.66 142.24)
 		)
 		(stroke
@@
 	(wire
 		(pts
-			(xy 185.42 72.39) (xy 191.77 72.39)
+			(xy 43.18 149.86) (xy 43.18 156.21)
 		)
 		(stroke
@@
 	(wire
 		(pts
-			(xy 77.47 71.12) (xy 78.74 71.12)
+			(xy 185.42 72.39) (xy 191.77 72.39)
 		)
 		(stroke
@@
 	(symbol
 		(lib_id "power:+5V")
-		(at 135.89 96.52 90)
+		(at 129.54 96.52 0)
 		(unit 1)
 		(exclude_from_sim no)
@@
 		(fields_autoplaced yes)
 		(property "Reference" "#PWR05"
-			(at 139.7 96.52 0)
+			(at 129.54 100.33 0)
 			(effects
 				(font
@@
 		)
 		(property "Value" "+5V"
-			(at 132.08 96.5199 90)
+			(at 129.54 91.44 0)
 			(effects
 				(font
 					(size 1.27 1.27)
 				)
-				(justify left)
 			)
 		)
 		(property "Footprint" ""
-			(at 135.89 96.52 0)
+			(at 129.54 96.52 0)
 			(effects
 				(font
@@
 		)
 		(property "Datasheet" ""
-			(at 135.89 96.52 0)
+			(at 129.54 96.52 0)
 			(effects
 				(font
@@
 		)
 		(property "Description" "Power symbol creates a global label with name \"+5V\""
-			(at 135.89 96.52 0)
+			(at 129.54 96.52 0)
 			(effects
 				(font
@@
 	(symbol
 		(lib_id "power:+5V")
-		(at 59.69 73.66 90)
+		(at 57.15 73.66 0)
 		(unit 1)
 		(exclude_from_sim no)
@@
 		(fields_autoplaced yes)
 		(property "Reference" "#PWR011"
-			(at 63.5 73.66 0)
+			(at 57.15 77.47 0)
 			(effects
 				(font
@@
 		)
 		(property "Value" "+5V"
-			(at 55.88 73.6599 90)
+			(at 57.15 68.58 0)
 			(effects
 				(font
 					(size 1.27 1.27)
 				)
-				(justify left)
 			)
 		)
 		(property "Footprint" ""
-			(at 59.69 73.66 0)
+			(at 57.15 73.66 0)
 			(effects
 				(font
@@
 		)
 		(property "Datasheet" ""
-			(at 59.69 73.66 0)
+			(at 57.15 73.66 0)
 			(effects
 				(font
@@
 		)
 		(property "Description" "Power symbol creates a global label with name \"+5V\""
-			(at 59.69 73.66 0)
+			(at 57.15 73.66 0)
 			(effects
 				(font
@@
 	(symbol
 		(lib_id "power:+5V")
-		(at 107.95 67.31 90)
+		(at 107.95 67.31 0)
 		(unit 1)
 		(exclude_from_sim no)
@@
 		(fields_autoplaced yes)
 		(property "Reference" "#PWR07"
-			(at 111.76 67.31 0)
+			(at 107.95 71.12 0)
 			(effects
 				(font
@@
 		)
 		(property "Value" "+5V"
-			(at 104.14 67.3099 90)
+			(at 107.95 62.23 0)
 			(effects
 				(font
 					(size 1.27 1.27)
 				)
-				(justify left)
 			)
 		)
